File: _pcb/LoRaProMini.kicad_pcb (KiCad board)
At the start: 2 copper layers, 0 parts

Commit message: Added the first PCB Layout
Parts:
- added 1-WIRE BUS: Conn_01x03, Connector_JST:JST_PH_B3B-PH-K_1x03_P2.00mm_Vertical, F.Cu at (184.9, 84.5)
- added ANT: Antenna_Shield, foorschtbar:Antenna_SMA_uFL, F.Cu at (103.4, 90.7)
- added C1: C, Capacitor_SMD:C_0805_2012Metric_Pad1.18x1.45mm_HandSolder, F.Cu at (130.9, 102.7)
- added C2: 1uF, Capacitor_SMD:C_0805_2012Metric_Pad1.18x1.45mm_HandSolder, F.Cu at (180.4, 103.6)
- added C3: 1uF, Capacitor_SMD:C_0805_2012Metric_Pad1.18x1.45mm_HandSolder, F.Cu at (175.4, 103.6)
- added C4: C, Capacitor_SMD:C_0805_2012Metric_Pad1.18x1.45mm_HandSolder, F.Cu at (170.4, 103.6)
- added C5: 1000uF, Capacitor_Tantalum_SMD:CP_EIA-7343-43_Kemet-X_Pad2.25x2.55mm_HandSolder, F.Cu at (170.4, 90.7)
- added DS18B20: DS18B20, Package_TO_SOT_THT:TO-92_Inline, F.Cu at (170.9, 81.2)
- added I2C BUS: Conn_01x04, Connector_JST:JST_PH_B4B-PH-K_1x04_P2.00mm_Vertical, F.Cu at (177.9, 87.7)
- added LoRa: RFM95W-868S2, foorschtbar:HOPERF_RFM9XW_SMD, F.Cu at (120.4, 90.7)
- added PWR: Conn_01x02, Connector_JST:JST_PH_B2B-PH-K_1x02_P2.00mm_Vertical, F.Cu at (184.9, 94.9)
- added R1: R, Resistor_SMD:R_0805_2012Metric_Pad1.20x1.40mm_HandSolder, F.Cu at (170.4, 97.6)
- added R2: R, Resistor_SMD:R_0805_2012Metric_Pad1.20x1.40mm_HandSolder, F.Cu at (170.4, 100.6)
- added R3: 4,7k, Resistor_SMD:R_0805_2012Metric_Pad1.20x1.40mm_HandSolder, F.Cu at (177.3, 83.2)
- added R4: 4,7k, Resistor_SMD:R_0805_2012Metric_Pad1.20x1.40mm_HandSolder, F.Cu at (177.3, 80.2)
- added R5: 4,7k, Resistor_SMD:R_0805_2012Metric_Pad1.20x1.40mm_HandSolder, F.Cu at (177.3, 77.2)
- added REF**: MountingHole_2.2mm_M2, MountingHole:MountingHole_2.2mm_M2, F.Cu at (185.4, 103.2)
- added REF**: MountingHole_2.2mm_M2, MountingHole:MountingHole_2.2mm_M2, F.Cu at (185.4, 78.2)
- added REF**: MountingHole_2.2mm_M2, MountingHole:MountingHole_2.2mm_M2, F.Cu at (102.4, 103.2)
- added REF**: MountingHole_2.2mm_M2, MountingHole:MountingHole_2.2mm_M2, F.Cu at (102.4, 78.2)
- added U1: MCP1700-3302E_SOT23, Package_TO_SOT_SMD:SOT-23_Handsoldering, F.Cu at (177.9, 99.1)
- added X1: ARDUINO_PRO_MINI, foorschtbar:Arduino_Pro_Mini, F.Cu at (149.4, 90.7)
Routing:
- net Net-(AE1-Pad1): track 0.00 -> 14.6 mm
- net GND: track 0.00 -> 3.80 mm, vias 0 -> 43
- added copper zone on B.Cu, net GND
- added copper zone on F.Cu, net GND
Other:
- board outline added: 90 x 32 mm

Commit message: Update PCB
Parts:
- added REF**: KiCad-Logo2_5mm_SilkScreen, Symbol:KiCad-Logo2_5mm_SilkScreen, B.Cu at (143.9, 90.7)
- Arduino Pro Mini: renamed from X1; value ARDUINO_PRO_MINI -> Arduino_Pro_Mini
- REF** (x4): value MountingHole_2.2mm_M2 -> MountingHole_2.2mm_M2_Pad_Via; footprint MountingHole:MountingHole_2.2mm_M2 -> MountingHole:MountingHole_2.2mm_M2_Pad_Via
- moved R2 3.05 mm to (170.2, 97.5)
- moved R1 3.01 mm to (170.2, 100.6)
- moved C1 1.01 mm to (130.4, 101.8), turned to 270 degrees
- moved C4 0.16 mm to (170.2, 103.6)
- moved I2C BUS 0.05 mm to (177.9, 87.7)
- turned R5 to 180 degrees
- turned R4 to 180 degrees
- renumbered LoRa to RFM95W
Connections:
- Arduino Pro Mini pad 1: (no net) -> Net-(X1-Pad1)
- Arduino Pro Mini pad 11: LORA_DIO2 -> LORA_DIO0
- Arduino Pro Mini pad 13: (no net) -> Net-(X1-Pad13)
- Arduino Pro Mini pad 15: (no net) -> Net-(X1-Pad15)
- Arduino Pro Mini pad 17: (no net) -> Net-(X1-Pad17)
- Arduino Pro Mini pad 18: (no net) -> Net-(X1-Pad18)
- Arduino Pro Mini pad 19: (no net) -> Net-(X1-Pad19)
- Arduino Pro Mini pad 2: (no net) -> Net-(X1-Pad2)
- Arduino Pro Mini pad 27: (no net) -> GND
- Arduino Pro Mini pad 28: (no net) -> Net-(X1-Pad28)
- Arduino Pro Mini pad 29: (no net) -> Net-(X1-Pad29)
- Arduino Pro Mini pad 3: (no net) -> Net-(X1-Pad3)
- Arduino Pro Mini pad 5: LORA_DIO0 -> LORA_DIO2
- Arduino Pro Mini pad 6: (no net) -> Net-(X1-Pad6)
- Arduino Pro Mini pad 7: (no net) -> Net-(X1-Pad7)
- Arduino Pro Mini pad 8: (no net) -> Net-(X1-Pad8)
- PWR pad 1: GND -> +BATT
- PWR pad 2: +BATT -> GND
- RFM95W pad 11: (no net) -> Net-(U2-Pad11)
- RFM95W pad 12: (no net) -> Net-(U2-Pad12)
- RFM95W pad 7: (no net) -> Net-(U2-Pad7)
Routing:
- net +3V3: track 0.00 -> 107.8 mm
- net 1-WIRE: track 0.00 -> 59.5 mm, vias 0 -> 1
- net MCU_SDA: track 0.00 -> 42.4 mm, vias 0 -> 2
- net MCU_SCL: track 0.00 -> 36.7 mm, vias 0 -> 2
- net LORA_DIO2: track 0.00 -> 36.3 mm
- net MCU_A0: track 0.00 -> 33.2 mm, vias 0 -> 2
- net SPI_SCK: track 0.00 -> 31.4 mm, vias 0 -> 1
- net SPI_CS_LORA: track 0.00 -> 26.7 mm, vias 0 -> 1
- net SPI_MOSI: track 0.00 -> 26.4 mm, vias 0 -> 1
- net SPI_MISO: track 0.00 -> 26.2 mm, vias 0 -> 1
- net LORA_DIO1: track 0.00 -> 25.6 mm
- net LORA_DIO0: track 0.00 -> 25.1 mm
- net +BATT: track 0.00 -> 20.9 mm, vias 0 -> 2
- net LORA_RST: track 0.00 -> 19.9 mm
- net GND: track 3.80 -> 3.94 mm, vias 43 -> 45
Other:
- board text added: "05/2021"
- board text added: "3.3V"
- board text added: "DATA"
- board text added: "GND"
- board text added: "JLCJLCJLCJLC"
- board text added: "LoRaProMini"
- board text added: "PCB v1.0"
- board text added: "SCL"
- board text added: "SDA"
- board text added: "VIN"
- board text added: "https://github.com/foorschtbar/LoRaProMini"
- board text added: "© 2021 foorschtbar"

Commit message: Updated PCB
Routing:
- net GND: vias 45 -> 46
