File: pcb/LoRaProMini.kicad_pcb (KiCad board)
At the start: 2 copper layers, 72 x 27 mm, 37 parts, among them J1 Conn_01x02, J2 Conn_01x03, J3 Conn_01x04, J4 Conn_01x05, J5 Conn_01x05, J6 Conn_01x08, J7 Conn_01x02, J8 Conn_01x02, SW1 SW_Push, U1 MCP1700-3302E_SOT23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

Commit message: Deploying to gh-pages from @ foorschtbar/LoRaProMini@a938d8310966b8f3c1edb3024db222770cf6ebb0 🚀
Other:
- board text added: "2021/10"
- board text added: "NODE ID"
- board text added: "REV 3.1"
- board text removed: "2021/09"
- board text removed: "REV 3.0"

Commit message: Fixed C7 (10uf --> 100nF)
Parts:
- AE1: footprint foorschtbar:Antenna_SMA_uFL -> Antenna_SMA_uFL:Antenna_SMA_uFL
- C7: value 10uF -> 100nf
- J5: footprint foorschtbar:Holes_1x05_P2.54mm -> Holes_1x05_P2.54mm:Holes_1x05_P2.54mm
- J6: footprint foorschtbar:Holes_1x08_P2.54mm -> Holes_1x08_P2.54mm:Holes_1x08_P2.54mm
- U2: footprint foorschtbar:HOPERF_RFM9XW_SMD -> HOPERF_RFM9XW_SMD:HOPERF_RFM9XW_SMD
- Y1: footprint Crystal:Resonator_SMD_muRata_CSTxExxV-3Pin_3.0x1.1mm -> Crystal:Resonator_SMD_Murata_CSTxExxV-3Pin_3.0x1.1mm
Connections:
- net +3V3 renamed +3.3V
- U2 pad 11: Net-(U2-Pad11) -> unconnected-(U2-DIO3-Pad11)
- U2 pad 12: Net-(U2-Pad12) -> unconnected-(U2-DIO4-Pad12)
- U2 pad 7: Net-(U2-Pad7) -> unconnected-(U2-DIO5-Pad7)
Routing:
- net +3.3V: track 172.4 -> 211.2 mm
- net GND: track 12.5 -> 9.74 mm, vias 54 -> 55
- net MCU_A0_BAT: track 21.8 -> 20.5 mm
- net MCU_D3: track 53.2 -> 52.4 mm
- net LORA_RST: track 21.3 -> 20.5 mm
Other:
- net class Default removed
- board text added: "2023/03"
- board text added: "REV 3.2"
- board text removed: "2021/10"
- board text removed: "REV 3.1"
